File: piboy.brd (EAGLE design)
At the start: 76.2 x 76.2 mm, 75 parts, among them CN4 MicroUSB, T1 MMUN2133LT1G, U1 TPS61090RSAR, U2 MCP73871

Commit message: -finished silkscreen -done before copper pours
Parts:
- renumbered LED1 to LBO, LED2 to ON
Other:
- board text added: "B"
- board text added: "C1"
- board text added: "C2"
- board text added: "C4"
- board text added: "C6"
- board text added: "C7"
- board text added: "C8"
- board text added: "G"
- board text added: "O"
- board text added: "R"
- board text added: "R1"
- board text added: "R13"
- board text added: "R14"
- board text added: "R16"
- board text added: "R17"
- board text added: "R2"
- board text added: "R20"
- board text added: "R3"
- board text added: "R5"
- board text added: "R6"
- board text added: "R7"
- board text added: "R8"
- board text added: "THRM"
Changed lines of the file:
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@@
 <layer number="14" name="Route14" color="1" fill="6" visible="no" active="no"/>
 <layer number="15" name="Route15" color="4" fill="6" visible="no" active="no"/>
-<layer number="16" name="Bottom" color="1" fill="1" visible="yes" active="yes"/>
+<layer number="16" name="Bottom" color="1" fill="1" visible="no" active="yes"/>
 <layer number="17" name="Pads" color="2" fill="1" visible="yes" active="yes"/>
 <layer number="18" name="Vias" color="2" fill="1" visible="yes" active="yes"/>
@@
 <text x="34.5" y="49.5" size="1.778" layer="26" font="vector" rot="MR270">C14</text>
 <text x="37.5" y="58.5" size="1.778" layer="26" font="vector" rot="MR0">R4</text>
+<text x="40.6" y="65.5" size="1.778" layer="26" font="vector" rot="MR0">R3</text>
+<text x="45.9" y="63.6" size="1.778" layer="26" font="vector" rot="MR0">C6</text>
+<text x="51.1" y="58.1" size="1.778" layer="26" font="vector" rot="MR0">C7</text>
+<text x="63.5" y="61.3" size="1.778" layer="26" font="vector" rot="MR0">THRM</text>
+<text x="62.3" y="57.8" size="1.778" layer="26" font="vector" rot="MR0">R14</text>
+<text x="64.4" y="54.4" size="1.778" layer="26" font="vector" rot="MR0">R8</text>
+<text x="61.3" y="48.8" size="1.778" layer="26" font="vector" rot="MR0">C8</text>
+<text x="65.4" y="49.7" size="1.778" layer="26" font="vector" rot="MR0">R6</text>
+<text x="57.2" y="49.3" size="1.778" layer="26" font="vector" rot="MR270">R17</text>
+<text x="54.9" y="49.6" size="1.778" layer="26" font="vector" rot="MR270">R16</text>
+<text x="52.1" y="47.4" size="1.778" layer="26" font="vector" rot="MR0">R2</text>
+<text x="47.8" y="46.3" size="1.778" layer="26" font="vector" rot="MR270">C1</text>
+<text x="43.4" y="50.8" size="1.778" layer="26" font="vector" rot="MR270">R13</text>
+<text x="45.8" y="54.3" size="1.778" layer="26" font="vector" rot="MR270">R1</text>
+<text x="49.2" y="54.8" size="1.778" layer="26" font="vector" rot="MR0">C4</text>
+<text x="73.2" y="51.9" size="1.778" layer="26" font="vector" rot="MR0">R7</text>
+<text x="72.5" y="55.5" size="1.778" layer="26" font="vector" rot="MR0">C2</text>
+<text x="74.5" y="58.5" size="1.778" layer="26" font="vector" rot="MR0">R20</text>
+<text x="68.3" y="62.5" size="1.778" layer="26" font="vector" rot="MR0">R5</text>
+<text x="74.6" y="63.3" size="1.778" layer="25" font="vector">B</text>
+<text x="71.4" y="60.5" size="1.778" layer="25" font="vector">R</text>
+<text x="71.4" y="57.3" size="1.778" layer="25" font="vector">O</text>
+<text x="73.4" y="53.9" size="1.778" layer="25" font="vector">G</text>
 </plain>
 <attributes>
@@
 <element name="DONE" library="piboy_new" package="ADAFRUIT_CHIPLED_0603" value="GREEN" x="74" y="56.3" rot="R90"/>
 <element name="L1" library="microbuilder" package="INDUCTOR_5X5MM_TDK_VLC5045" value="6.8uH" x="7" y="38.71" rot="MR0"/>
-<element name="LED1" library="piboy_new" package="ADAFRUIT_CHIPLED_0603" value="RED" x="74" y="61.3" rot="R270"/>
-<element name="LED2" library="piboy_new" package="ADAFRUIT_CHIPLED_0603" value="BLUE" x="74" y="62.7" rot="R270"/>
+<element name="LBO" library="piboy_new" package="ADAFRUIT_CHIPLED_0603" value="RED" x="74" y="61.3" rot="R270"/>
+<element name="ON" library="piboy_new" package="ADAFRUIT_CHIPLED_0603" value="BLUE" x="74" y="62.7" rot="R270"/>
 <element name="R1" library="adafruit" package="R0805" value="1.87M" x="46.94" y="52.1" rot="MR270"/>
 <element name="R13" library="adafruit" package="R0805" value="200K" x="44.59" y="47.99" rot="MR270"/>
@@
 <contactref element="C2" pad="2"/>
 <contactref element="C6" pad="2"/>
-<contactref element="LED2" pad="C"/>
+<contactref element="ON" pad="C"/>
 <contactref element="R2" pad="1"/>
-<contactref element="LED1" pad="C"/>
+<contactref element="LBO" pad="C"/>
 <contactref element="R7" pad="2"/>
 <contactref element="C7" pad="2"/>
@@
 </signal>
 <signal name="N$2">
-<contactref element="LED1" pad="A"/>
+<contactref element="LBO" pad="A"/>
 <contactref element="R20" pad="1"/>
 <wire x1="68.89" y1="59.23" x2="71.18" y2="59.23" width="0.1524" layer="16"/>
@@
 <signal name="N$4">
 <contactref element="R5" pad="2"/>
-<contactref element="LED2" pad="A"/>
+<contactref element="ON" pad="A"/>
 <wire x1="66.97" y1="61.36" x2="67.3967125" y2="61.36" width="0.1524" layer="16"/>
 <wire x1="67.3967125" y1="61.36" x2="68.3253125" y2="62.2886" width="0.1524" layer="16"/>
